File: PCB/PCB.kicad_pcb (KiCad board)
At the start: 2 copper layers, 100 x 100 mm, 48 parts, among them J1 Conn_01x04, J10 Conn_01x02, J11 Conn_01x02, J12 Conn_01x02, J13 Conn_01x02, J14 Conn_01x02, J2 Conn_01x04, J3 Conn_01x04, J4 Conn_01x04, J5 Conn_01x04, J6 Conn_01x04, J7 Conn_01x02, J8 Conn_01x02, J9 Conn_01x02, U1 MAX3485, U2 ESP32-DevKitC, U3 INA226, U4 INA226, U5 PCA9685PW, U6 TSR_1-2450, U7 AMS1117-3.3, U8 LM75B

Commit message: Updated PCB
Parts:
- added J16: Conn_01x12, Connector_PinHeader_2.54mm:PinHeader_1x12_P2.54mm_Vertical, F.Cu at (144.8, 137.2)
- added J17: Conn_01x12, Connector_PinHeader_2.54mm:PinHeader_1x12_P2.54mm_Vertical, F.Cu at (142.2, 137.2)
- added J18: Conn_01x12, Connector_PinHeader_2.54mm:PinHeader_1x12_P2.54mm_Vertical, F.Cu at (139.7, 137.2)
- added R8: 2m, Resistor_SMD:R_2512_6332Metric_Pad1.40x3.35mm_HandSolder, F.Cu at (112.3, 138.3)
Routing:
- net GND: track 0.00 -> 50.0 mm, vias 0 -> 3
- net Net-(D8-K): track 0.00 -> 46.4 mm
- net /485_P: track 0.00 -> 45.0 mm
- net /485_N: track 0.00 -> 45.0 mm
- net +5V: track 0.00 -> 22.0 mm
- net Net-(D10-A): track 0.00 -> 18.6 mm
- net +3V3: track 0.00 -> 11.8 mm, vias 0 -> 5
- net +3s_LIPO: vias 0 -> 32
- added copper zone on In2.Cu, net +3V3
- added copper zone on B.Cu, net +3s_LIPO
- added copper zone on F.Cu, net +3s_LIPO
- added copper zone on F.Cu, net +3s_LIPO_EXT
- added copper zone on B.Cu, net +5s_LIPO
- added copper zone on F.Cu, net GND
- added copper zone on In1.Cu, net GND
Other:
- copper layers 2 -> 4
