File: PCB/PCB.kicad_sch (KiCad schematic)
At the start: 2 parts, among them U1 MAX485E, U2 ESP32-DevKitC

Commit message: Updated PCB
Parts:
- removed U1: MAX485E, Package_SO:SOIC-8_3.9x4.9mm_P1.27mm, symbol Interface_UART:MAX485E
- added D1, D2, D3, D5, D6, D7: LED, LED_THT:LED_D5.0mm, symbol Device:LED
- added D10, D8, D9: 1N5822, Diode_THT:D_DO-201AD_P15.24mm_Horizontal, symbol Diode:1N5822
- added D4: SM712_SOT23, Package_TO_SOT_SMD:SOT-23, symbol Diode:SM712_SOT23
- added J1, J2, J3, J4, J5, J6: Conn_01x04, Connector_JST:JST_ZH_B4B-ZR_1x04_P1.50mm_Vertical, symbol Connector_Generic:Conn_01x04
- added J10, J11, J12, J13, J14, J9: Conn_01x02, Connector_JST:JST_XH_B2B-XH-AM_1x02_P2.50mm_Vertical, symbol Connector_Generic:Conn_01x02
- added J7, J8: Conn_01x02, Connector_AMASS:AMASS_XT60-M_1x02_P7.20mm_Vertical, symbol Connector_Generic:Conn_01x02
- added R1, R2, R3: 1000, Resistor_THT:R_Axial_DIN0207_L6.3mm_D2.5mm_P10.16mm_Horizontal, symbol Device:R
- added R10, R5, R6, R9: 4k7, Resistor_THT:R_Axial_DIN0207_L6.3mm_D2.5mm_P10.16mm_Horizontal, symbol Device:R
- added R11, R12, R13: 300, Resistor_THT:R_Axial_DIN0207_L6.3mm_D2.5mm_P10.16mm_Horizontal, symbol Device:R
- added R4: 120, Resistor_THT:R_Axial_DIN0207_L6.3mm_D2.5mm_P10.16mm_Horizontal, symbol Device:R
- added R7, R8: TBD, symbol Device:R
- added TP1, TP2, TP3, TP4: TestPoint, TestPoint:TestPoint_Pad_D2.0mm, symbol Connector:TestPoint
- added TP5: TestPoint, TestPoint:TestPoint_Pad_2.0x2.0mm, symbol Connector:TestPoint
- added U1: MAX3485, Package_SO:SOIC-8_3.9x4.9mm_P1.27mm, symbol Interface_UART:MAX3485
- added U3, U4: INA226, Package_SO:TSSOP-10_3x3mm_P0.5mm, symbol Sensor_Energy:INA226
- added U5: PCA9685PW, Package_SO:TSSOP-28_4.4x9.7mm_P0.65mm, symbol Driver_LED:PCA9685PW
- added U6: TSR_1-2450, Converter_DCDC:Converter_DCDC_TRACO_TSR-1_THT, symbol Converter_DCDC:TSR_1-2450
- added U7: AMS1117-3.3, Package_TO_SOT_SMD:SOT-223-3_TabPin2, symbol Regulator_Linear:AMS1117-3.3
- added U8: LM75B, Package_SO:SOIC-8_3.9x4.9mm_P1.27mm, symbol Sensor_Temperature:LM75B
Connections:
- net STAT_LED_2: now reaches U2.10 (DAC_2/ADC2_CH9/GPIO26)
- net STAT_LED_2: now also D7.1 (K)
- net GND: now reaches U2.14 (GND), U2.32 (GND), U2.38 (GND)
- net GND: now also D4.3 (common), D5.1 (K), J1.4 (Pin_4), J10.1 (Pin_1), J11.1 (Pin_1), J12.1 (Pin_1), J13.1 (Pin_1), J14.1 (Pin_1), J2.4 (Pin_4), J3.4 (Pin_4), J4.4 (Pin_4), J5.4 (Pin_4), J6.4 (Pin_4), J7.2 (Pin_2), J8.2 (Pin_2), J9.1 (Pin_1), R6.1, TP5.1, U1.5 (GND), U3.7 (GND), U4.2 (A0), U4.7 (GND), U5.1 (A0), U5.14 (VSS), U5.2 (A1), U5.24 (A5), U5.25 (EXTCLK), U5.3 (A2), U5.4 (A3), U5.5 (A4), U6.2 (GND), U7.1 (GND), U8.4 (GND), U8.5 (A2), U8.6 (A1), U8.7 (A0)
- net +5V: now reaches U2.19 (5V)
- net +5V: now also D10.1 (K), TP2.1, U7.3 (VI)
- net TX_485_EN: now reaches U2.29 (GPIO5)
- net TX_485_EN: now also D3.1 (K), U1.2 (~{RE}), U1.3 (DE)
- net RXD_485: now reaches U2.30 (GPIO18)
- net RXD_485: now also D1.1 (K), U1.1 (RO)
- net TXD_485: now reaches U2.31 (GPIO19)
- net TXD_485: now also D2.1 (K), U1.4 (DI)
- net SDA: now reaches U2.33 (GPIO21)
- net SDA: now also R9.1, U3.4 (SDA), U4.4 (SDA), U5.27 (SDA), U8.1 (SDA)
- net SCL: now reaches U2.36 (GPIO22)
- net SCL: now also R10.1, U3.5 (SCL), U4.5 (SCL), U5.26 (SCL), U8.2 (SCL)
- net SERVO_EN: now reaches U2.37 (GPIO23)
- net SERVO_EN: now also U5.23 (~{OE})
- net STAT_LED_1: now reaches U2.9 (DAC_1/ADC2_CH8/GPIO25)
- net STAT_LED_1: now also D6.1 (K)
- new net: D2.2 (A), R2.2
- new net: D7.2 (A), R13.2
- new net: D8.1 (K), D9.1 (K), U6.1 (Vin)
- new net: D10.2 (A), U6.3 (Vout)
- new net: D1.2 (A), R1.2
- new net: D6.2 (A), R12.2
- new net: D3.2 (A), R3.2
- new net: D5.2 (A), R11.2
- new net +3V3: R1.1, R10.2, R11.1, R12.1, R13.1, R2.1, R3.1, R5.2, R9.2, TP1.1, U1.8 (VCC), U3.1 (A1), U3.2 (A0), U3.6 (VS), U4.1 (A1), U4.6 (VS), U5.28 (VDD), U7.2 (VO), U8.8 (+Vs)
- new net +3s_LIPO: D9.2 (A), R8.1, U4.9 (Vin-)
- new net +3s_LIPO_EXT: J8.1 (Pin_1), R8.2, TP4.1, U4.10 (Vin+), U4.8 (Vbus)
- new net +5s_LIPO: D8.2 (A), J10.2 (Pin_2), J11.2 (Pin_2), J12.2 (Pin_2), J13.2 (Pin_2), J14.2 (Pin_2), J9.2 (Pin_2), R7.1, U3.9 (Vin-)
- new net +5s_LIPO_EXT: J7.1 (Pin_1), R7.2, TP3.1, U3.10 (Vin+), U3.8 (Vbus)
- new net 485_N: D4.2 (A2), J1.2 (Pin_2), J2.2 (Pin_2), J3.2 (Pin_2), J4.2 (Pin_2), J5.2 (Pin_2), J6.2 (Pin_2), R4.1, R6.2, U1.7 (B)
- new net 485_P: D4.1 (A1), J1.3 (Pin_3), J2.3 (Pin_3), J3.3 (Pin_3), J4.3 (Pin_3), J5.3 (Pin_3), J6.3 (Pin_3), R4.2, R5.1, U1.6 (A)
- new net SERVO_1: U5.6 (LED0)
- new net SERVO_10: U5.16 (LED9)
- new net SERVO_11: U5.17 (LED10)
- new net SERVO_12: U5.18 (LED11)
- new net SERVO_2: U5.7 (LED1)
- new net SERVO_3: U5.8 (LED2)
- new net SERVO_4: U5.9 (LED3)
- new net SERVO_5: U5.10 (LED4)
- new net SERVO_6: U5.11 (LED5)
- new net SERVO_7: U5.12 (LED6)
- new net SERVO_8: U5.13 (LED7)
- new net SERVO_9: U5.15 (LED8)
- no-connect marks 0 -> 39
Other:
- note added: "Diagnostic LEDs"
- note added: "GND testpoint"
- note added: "I2C pull ups"
- note added: "Power monitoring"
- note added: "Power supplies"
- note added: "RS485 - Motors"
- note added: "Servo controller"
- note added: "Temperature sensor"
- moved on the sheet: U2

Commit message: Updated PCB
Parts:
- added J16, J17, J18: Conn_01x12, Connector_PinHeader_2.54mm:PinHeader_1x12_P2.54mm_Vertical, symbol Connector_Generic:Conn_01x12
- R7, R8: value TBD -> 2m; footprint (none) -> Resistor_SMD:R_2512_6332Metric_Pad1.40x3.35mm_HandSolder
Connections:
- net +3s_LIPO: now also J17.1 (Pin_1), J17.10 (Pin_10), J17.11 (Pin_11), J17.12 (Pin_12), J17.2 (Pin_2), J17.3 (Pin_3), J17.4 (Pin_4), J17.5 (Pin_5), J17.6 (Pin_6), J17.7 (Pin_7), J17.8 (Pin_8), J17.9 (Pin_9)
- net GND: now also J16.1 (Pin_1), J16.10 (Pin_10), J16.11 (Pin_11), J16.12 (Pin_12), J16.2 (Pin_2), J16.3 (Pin_3), J16.4 (Pin_4), J16.5 (Pin_5), J16.6 (Pin_6), J16.7 (Pin_7), J16.8 (Pin_8), J16.9 (Pin_9)
- net SERVO_1: now also J18.1 (Pin_1)
- net SERVO_10: now also J18.10 (Pin_10)
- net SERVO_11: now also J18.11 (Pin_11)
- net SERVO_12: now also J18.12 (Pin_12)
- net SERVO_2: now also J18.2 (Pin_2)
- net SERVO_3: now also J18.3 (Pin_3)
- net SERVO_4: now also J18.4 (Pin_4)
- net SERVO_5: now also J18.5 (Pin_5)
- net SERVO_6: now also J18.6 (Pin_6)
- net SERVO_7: now also J18.7 (Pin_7)
- net SERVO_8: now also J18.8 (Pin_8)
- net SERVO_9: now also J18.9 (Pin_9)
